File: pcb/daydream.kicad_sch (KiCad schematic)
At the start: 1 part

Commit message: finished the schematic
Parts:
- added D1, D2: LED, symbol Device:LED
- added R1, R2: 200ohm, symbol Device:R
- added SW1, SW2: SW_Push, symbol Switch:SW_Push
Connections:
- net at BT1.1 (+): now also R1.1, R2.1
- net GND: now reaches BT1.2 (-)
- net GND: now also D1.1 (K), D2.1 (K)
- new net: D1.2 (A), R2.2
- new net: D2.2 (A), R1.2
- no-connect marks 0 -> 4

Commit message: added uhh a lot of stuff
Parts:
- BT1: footprint (none) -> Battery:BatteryHolder_Keystone_3000_1x12mm
- D1, D2: footprint (none) -> LED_THT:LED_D5.0mm
- R1, R2: footprint (none) -> Resistor_THT:R_Axial_DIN0207_L6.3mm_D2.5mm_P7.62mm_Horizontal
- SW1, SW2: footprint (none) -> Button_Switch_THT:SW_PUSH_6mm_H5mm
Changed lines of the file:
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@@
 			)
 		)
-		(property "Footprint" ""
+		(property "Footprint" "Battery:BatteryHolder_Keystone_3000_1x12mm"
 			(at 58.166 97.79 90)
 			(effects
@@
 			)
 		)
-		(property "Footprint" ""
+		(property "Footprint" "Resistor_THT:R_Axial_DIN0207_L6.3mm_D2.5mm_P7.62mm_Horizontal"
 			(at 37.592 109.22 90)
 			(effects
@@
 			)
 		)
-		(property "Footprint" ""
+		(property "Footprint" "Button_Switch_THT:SW_PUSH_6mm_H5mm"
 			(at 96.52 111.76 0)
 			(effects
@@
 			)
 		)
-		(property "Footprint" ""
+		(property "Footprint" "LED_THT:LED_D5.0mm"
 			(at 58.42 114.3 0)
 			(effects
@@
 			)
 		)
-		(property "Footprint" ""
+		(property "Footprint" "LED_THT:LED_D5.0mm"
 			(at 45.72 119.38 0)
 			(effects
@@
 			)
 		)
-		(property "Footprint" ""
+		(property "Footprint" "Button_Switch_THT:SW_PUSH_6mm_H5mm"
 			(at 96.52 124.46 0)
 			(effects
@@
 			)
 		)
-		(property "Footprint" ""
+		(property "Footprint" "Resistor_THT:R_Axial_DIN0207_L6.3mm_D2.5mm_P7.62mm_Horizontal"
 			(at 49.022 106.68 90)
 			(effects
